Commit message: simplify collision shapes by mergin stl

File: wolfgang_description/urdf/robot.urdf (robot description, URDF)
Before this commit: robot wolfgang, 45 links, 44 joints
Links:
- link head: geometry collision mesh filename=package://head.stl; visual mesh filename=package://head.stl
- link l_ankle: geometry collision mesh filename=package://l_ankle.stl; visual mesh filename=package://l_ankle.stl
- link l_foot: geometry collision mesh filename=package://l_foot.stl; visual mesh filename=package://l_foot.stl
- link l_hip_1: geometry collision mesh filename=package://l_hip_1.stl; visual mesh filename=package://l_hip_1.stl
- link l_hip_2: geometry collision mesh filename=package://l_hip_2.stl; visual mesh filename=package://l_hip_2.stl
- link l_lower_arm: geometry collision mesh filename=package://l_lower_arm.stl; visual mesh filename=package://l_lower_arm.stl
- link l_lower_leg: geometry collision mesh filename=package://l_lower_leg.stl; visual mesh filename=package://l_lower_leg.stl
- link l_shoulder: geometry collision mesh filename=package://l_shoulder.stl; visual mesh filename=package://l_shoulder.stl
- link l_upper_arm: geometry collision mesh filename=package://l_upper_arm.stl; visual mesh filename=package://l_upper_arm.stl
- link l_upper_leg: geometry collision mesh filename=package://l_upper_leg.stl; visual mesh filename=package://l_upper_leg.stl
- link llb: geometry collision mesh filename=package://llb.stl; visual mesh filename=package://llb.stl
- link llf: geometry collision mesh filename=package://llf.stl; visual mesh filename=package://llf.stl
- link lrb: geometry collision mesh filename=package://lrb.stl; visual mesh filename=package://lrb.stl
- link lrf: geometry collision mesh filename=package://lrf.stl; visual mesh filename=package://lrf.stl
- link neck: geometry collision mesh filename=package://neck.stl; visual mesh filename=package://neck.stl
- link r_ankle: geometry collision mesh filename=package://r_ankle.stl; visual mesh filename=package://r_ankle.stl
- link r_foot: geometry collision mesh filename=package://r_foot.stl; visual mesh filename=package://r_foot.stl
- link r_hip_1: geometry collision mesh filename=package://r_hip_1.stl; visual mesh filename=package://r_hip_1.stl
- link r_hip_2: geometry collision mesh filename=package://r_hip_2.stl; visual mesh filename=package://r_hip_2.stl
- link r_lower_arm: geometry collision mesh filename=package://r_lower_arm.stl; visual mesh filename=package://r_lower_arm.stl
- link r_lower_leg: geometry collision mesh filename=package://r_lower_leg.stl; visual mesh filename=package://r_lower_leg.stl
- link r_shoulder: geometry collision mesh filename=package://r_shoulder.stl; visual mesh filename=package://r_shoulder.stl
- link r_upper_arm: geometry collision mesh filename=package://r_upper_arm.stl; visual mesh filename=package://r_upper_arm.stl
- link r_upper_leg: geometry collision mesh filename=package://r_upper_leg.stl; visual mesh filename=package://r_upper_leg.stl
- link rlb: geometry collision mesh filename=package://rlb.stl; visual mesh filename=package://rlb.stl
- link rlf: geometry collision mesh filename=package://rlf.stl; visual mesh filename=package://rlf.stl
- link rrb: geometry collision mesh filename=package://rrb.stl; visual mesh filename=package://rrb.stl
- link rrf: geometry collision mesh filename=package://rrf.stl; visual mesh filename=package://rrf.stl
- link torso: geometry collision mesh filename=package://torso.stl; visual mesh filename=package://torso.stl

Commit message: Fixed some problems with robotis op2

File: wolfgang_description/urdf/robot.urdf (robot description, URDF)
Before this commit: robot wolfgang, 48 links, 47 joints
Joints:
- joint r_wrist_frame: origin xyz=3.1225e-16 -0.226182 -0.0235 rpy=1.5708 7.31053e-15 -1.5708 -> xyz=3.1225e-16 -0.226182 -0.0235 rpy=-1.5708 7.31053e-15 -1.5708

Commit message: Undo mistake in wolfgang urdf

File: wolfgang_description/urdf/robot.urdf (robot description, URDF)
Before this commit: robot wolfgang, 48 links, 47 joints
Joints:
- joint r_wrist_frame: origin xyz=3.1225e-16 -0.226182 -0.0235 rpy=-1.5708 7.31053e-15 -1.5708 -> xyz=3.1225e-16 -0.226182 -0.0235 rpy=1.5708 7.31053e-15 -1.5708

Commit message: new export from onshape, fix hip pitch limits

File: wolfgang_description/urdf/robot.urdf (robot description, URDF)
Before this commit: robot wolfgang, 48 links, 47 joints
Joints:
- joint LHipPitch: limit lower=-0.785398 upper=1.5708 effort=7.57 velocity=8.22 -> lower=-1.91986 upper=2.0944 effort=7.57 velocity=8.22
- joint RAnklePitch: origin xyz=-2.08167e-17 0.0505 -0.17 rpy=-1.5708 0.0364674 1.18307e-15 -> xyz=-1.38778e-17 0.0505 -0.17 rpy=-1.5708 0.0364674 1.18307e-15
- joint RHipPitch: limit lower=-1.5708 upper=0.785398 effort=7.57 velocity=8.22 -> lower=-2.0944 upper=1.91986 effort=7.57 velocity=8.22

Commit message: various fixes

File: wolfgang_description/urdf/robot.urdf (robot description, URDF)
Before this commit: robot wolfgang, 48 links, 47 joints
Joints:
- joint LAnklePitch: limit lower=-1.22173 upper=1.5708 effort=7.57 velocity=8.22 -> lower=-1.22173 upper=1.74533 effort=7.57 velocity=8.22
- joint RAnklePitch: limit lower=-1.5708 upper=1.22173 effort=7.57 velocity=8.22 -> lower=-1.74533 upper=1.22173 effort=7.57 velocity=8.22

Commit message: Remove camera optical frame from urdf.

File: wolfgang_description/urdf/robot.urdf (robot description, URDF)
Before this commit: robot wolfgang, 48 links, 47 joints
Links:
- removed link camera_optical_frame
Joints:
- removed joint camera_optical_frame_frame

Commit message: Add nubots legs to robot model

File: wolfgang_description/urdf/robot.urdf (robot description, URDF)
Before this commit: robot wolfgang, 47 links, 46 joints
Links:
- removed link l_ankle
- removed link l_cleat_l_back
- removed link l_cleat_l_front
- removed link l_cleat_r_back
- removed link l_cleat_r_front
- removed link l_foot
- removed link l_lower_leg
- removed link l_toe
- removed link llb
- removed link llf
- removed link lrb
- removed link lrf
- removed link r_ankle
- removed link r_cleat_l_back
- removed link r_cleat_l_front
- removed link r_cleat_r_back
- removed link r_cleat_r_front
- removed link r_foot
- removed link r_lower_leg
- removed link r_toe
- removed link rlb
- removed link rlf
- removed link rrb
- removed link rrf
- added link left_ankle; collision box size=0.04 0.08 0.065; visual box size=0.04 0.08 0.065
- added link left_foot [foot]; collision box size=0.125 0.0175 0.0585; collision box size=0.125 0.08 0.05
- added link left_lower_leg; collision box size=0.005 0.065 0.065; collision box size=0.005 0.065 0.065
- added link left_touch_sensor_bl; collision cylinder length=0.001 radius=0.009; collision sphere radius=0.009
- added link left_touch_sensor_br; collision cylinder length=0.001 radius=0.009; collision sphere radius=0.009
- added link left_touch_sensor_fl; collision cylinder length=0.001 radius=0.009; collision sphere radius=0.009
- added link left_touch_sensor_fr; collision cylinder length=0.001 radius=0.009; collision sphere radius=0.009
- added link right_ankle; collision box size=0.04 0.08 0.065; visual box size=0.04 0.08 0.065
- added link right_foot [foot]; collision box size=0.125 0.0175 0.0585; collision box size=0.125 0.08 0.05
- added link right_lower_leg; collision box size=0.005 0.065 0.065; collision box size=0.005 0.065 0.065
- added link right_touch_sensor_bl; collision cylinder length=0.001 radius=0.009; collision sphere radius=0.009
- added link right_touch_sensor_br; collision cylinder length=0.001 radius=0.009; collision sphere radius=0.009
- added link right_touch_sensor_fl; collision cylinder length=0.001 radius=0.009; collision sphere radius=0.009
- added link right_touch_sensor_fr; collision cylinder length=0.001 radius=0.009; collision sphere radius=0.009
- link l_sole: mass 1e-09 -> None
- link l_upper_leg: mass 0.242311 -> None; geometry collision box size=0.005 0.065 0.05; collision box size=0.005 0.065 0.05
- link r_sole: mass 1e-09 -> None
- link r_upper_leg: mass 0.242311 -> None; geometry collision box size=0.005 0.065 0.05; collision box size=0.005 0.065 0.05
Joints:
- removed joint LAnklePitch
- removed joint LAnkleRoll
- removed joint LHipPitch
- removed joint LHipRoll
- removed joint LHipYaw
- removed joint LKnee
- removed joint LLB
- removed joint LLF
- removed joint LRB
- removed joint LRF
- removed joint RAnklePitch
- removed joint RAnkleRoll
- removed joint RHipPitch
- removed joint RHipRoll
- removed joint RHipYaw
- removed joint RKnee
- removed joint RLB
- removed joint RLF
- removed joint RRB
- removed joint RRF
- removed joint l_cleat_l_back_frame
- removed joint l_cleat_l_front_frame
- removed joint l_cleat_r_back_frame
- removed joint l_cleat_r_front_frame
- removed joint l_toe_frame
- removed joint r_cleat_l_back_frame
- removed joint r_cleat_l_front_frame
- removed joint r_cleat_r_back_frame
- removed joint r_cleat_r_front_frame
- removed joint r_toe_frame
- added joint left_ankle_pitch: type revolute, parent left_lower_leg, child left_ankle, origin xyz=0 0.00001 -0.209753 rpy=-3.061991 0 -3.141591, axis -1 -0.000002 0, limit lower=-1.7 upper=1.7 effort=10 velocity=5.76
- added joint left_ankle_roll: type revolute, parent left_ankle, child left_foot [foot], origin xyz=0 0.04 0 rpy=-3.141591 -0.000005 -3.141591, axis 0.000002 -1 0.000002, limit lower=-1.5 upper=1.5 effort=10 velocity=5.76
- added joint left_foot [foot]_left_touch_sensor_bl_joint: type fixed, parent left_foot [foot], child left_touch_sensor_bl, origin xyz=0.057001 0.025012 -0.06106 rpy=0 0 0
- added joint left_foot [foot]_left_touch_sensor_br_joint: type fixed, parent left_foot [foot], child left_touch_sensor_br, origin xyz=-0.040999 0.025013 -0.061061 rpy=0 0 0
- added joint left_foot [foot]_left_touch_sensor_fl_joint: type fixed, parent left_foot [foot], child left_touch_sensor_fl, origin xyz=0.056999 -0.154145 -0.061056 rpy=0 0 0
- added joint left_foot [foot]_left_touch_sensor_fr_joint: type fixed, parent left_foot [foot], child left_touch_sensor_fr, origin xyz=-0.041001 -0.154153 -0.061058 rpy=0 0 0
- added joint left_knee_pitch: type revolute, parent left_upper_leg, child left_lower_leg, origin xyz=0 0.00924 -0.184766 rpy=0.046837 0 0, axis 1 0 0, limit lower=-0.3 upper=2.5 effort=10 velocity=5.76
- added joint right_ankle_pitch: type revolute, parent right_lower_leg, child right_ankle, origin xyz=0 0.00001 -0.19975 rpy=-3.064387 0 -3.141591, axis -1 -0.000002 0, limit lower=-1.7 upper=1.7 effort=10 velocity=5.76
- added joint right_ankle_roll: type revolute, parent right_ankle, child right_foot [foot], origin xyz=0 0.04 0 rpy=-3.141591 0.000004 -3.141591, axis 0.000002 -1 0.000002, limit lower=-1.5 upper=1.5 effort=10 velocity=5.76
- added joint right_foot [foot]_right_touch_sensor_bl_joint: type fixed, parent right_foot [foot], child right_touch_sensor_bl, origin xyz=0.041001 0.025012 -0.061061 rpy=0 0 0
- added joint right_foot [foot]_right_touch_sensor_br_joint: type fixed, parent right_foot [foot], child right_touch_sensor_br, origin xyz=-0.057499 0.025012 -0.061062 rpy=0 0 0
- added joint right_foot [foot]_right_touch_sensor_fl_joint: type fixed, parent right_foot [foot], child right_touch_sensor_fl, origin xyz=0.040899 -0.154143 -0.061056 rpy=0 0 0
- added joint right_foot [foot]_right_touch_sensor_fr_joint: type fixed, parent right_foot [foot], child right_touch_sensor_fr, origin xyz=-0.0575 -0.154151 -0.061058 rpy=0 0 0
- added joint right_knee_pitch: type revolute, parent right_upper_leg, child right_lower_leg, origin xyz=0 0.01024 -0.204744 rpy=0.045988 0 0, axis 1 0 0, limit lower=-0.3 upper=2.5 effort=10 velocity=5.76
- joint l_sole_frame: origin xyz=-0.0152219 0.0907683 -0.0529 rpy=-5.77818e-15 -6.98371e-15 1.5708 -> xyz=0.0 -0.05 -0.062 rpy=0.0 0.0 -1.5708; parent l_foot -> left_foot [foot]
- joint r_sole_frame: origin xyz=0.0152219 0.0907683 -0.0529 rpy=-4.1858e-16 2.36866e-15 1.5708 -> xyz=0.0 -0.05 -0.062 rpy=0.0 0.0 -1.5708; parent r_foot -> right_foot [foot]

Commit message: Some improvements

File: wolfgang_description/urdf/robot.urdf (robot description, URDF)
Before this commit: robot wolfgang, 37 links, 30 joints
Joints:
- removed joint left_ankle_pitch
- removed joint left_ankle_roll
- removed joint left_knee_pitch
- removed joint right_ankle_pitch
- removed joint right_ankle_roll
- removed joint right_knee_pitch
- added joint LAnklePitch: type revolute, parent left_lower_leg, child left_ankle, origin xyz=0 0.00001 -0.209753 rpy=-3.061991 0 -3.141591, axis -1 -0.000002 0, limit lower=-1.7 upper=1.7 effort=10 velocity=5.76
- added joint LAnkleRoll: type revolute, parent left_ankle, child left_foot [foot], origin xyz=0 0.04 0 rpy=-3.141591 -0.000005 -3.141591, axis 0.000002 -1 0.000002, limit lower=-1.5 upper=1.5 effort=10 velocity=5.76
- added joint LHipPitch: type revolute, parent l_hip_2, child l_upper_leg, origin xyz=0.026 6.93889e-18 -0.0691 rpy=2.67116e-16 -1.5708 0.0, axis 7.95491e-17 -3.00167e-16 -1.0, limit lower=-1.91986 upper=2.0944 effort=10 velocity=5.76
- added joint LHipRoll: type revolute, parent l_hip_1, child l_hip_2, origin xyz=-0.046 0.0414 6.93889e-18 rpy=3.14159 1.5708 0.0, axis -0.0 -0.0 -1.0, limit lower=-1.5708 upper=1.5708 effort=10 velocity=5.76
- added joint LHipYaw: type revolute, parent torso, child l_hip_1, origin xyz=1.82493e-15 0.055 -4.22839e-18 rpy=-1.5708 -0.0 0.0, axis -0.0 1.0 -0.0, limit lower=-1.5708 upper=1.5708 effort=10 velocity=5.76
- added joint LKnee: type revolute, parent l_upper_leg, child left_lower_leg, origin xyz=0 0.00924 -0.184766 rpy=0.046837 0 0, axis 1 0 0, limit lower=-0.3 upper=2.5 effort=10 velocity=5.76
- added joint RAnklePitch: type revolute, parent right_lower_leg, child right_ankle, origin xyz=0 0.00001 -0.19975 rpy=-3.064387 0 -3.141591, axis -1 -0.000002 0, limit lower=-1.7 upper=1.7 effort=10 velocity=5.76
- added joint RAnkleRoll: type revolute, parent right_ankle, child right_foot [foot], origin xyz=0 0.04 0 rpy=-3.141591 0.000004 -3.141591, axis 0.000002 -1 0.000002, limit lower=-1.5 upper=1.5 effort=10 velocity=5.76
- added joint RHipPitch: type revolute, parent r_hip_2, child r_upper_leg, origin xyz=-0.0265 -9.71445e-17 -0.0691 rpy=-1.5708 1.5708 0.0, axis -0.0 1.0 -0.0, limit lower=-2.0944 upper=1.91986 effort=10 velocity=5.76
- added joint RHipRoll: type revolute, parent r_hip_1, child r_hip_2, origin xyz=-0.046 0.0414 6.93889e-18 rpy=-3.14159 1.5708 0.0, axis -0.0 -0.0 -1.0, limit lower=-1.5708 upper=1.5708 effort=10 velocity=5.76
- added joint RHipYaw: type revolute, parent torso, child r_hip_1, origin xyz=7.99361e-15 -0.055 4.68375e-17 rpy=-1.5708 -0.0 0.0, axis -0.0 1.0 -0.0, limit lower=-1.5708 upper=1.5708 effort=10 velocity=5.76
- added joint RKnee: type revolute, parent r_upper_leg, child right_lower_leg, origin xyz=0 0.01024 -0.204744 rpy=0.045988 0 0, axis 1 0 0, limit lower=-0.3 upper=2.5 effort=10 velocity=5.76
